File: 4028-Series BCD-to-Decimal Decoder Tester.kicad_sch (KiCad schematic)
At the start: 33 parts, among them J1 USB_C_Receptacle_USB2.0, SW1 SW_Push, SW2 2MS1T2B2VS2QES, SW3 2MS1T2B2VS2QES, SW4 2MS1T2B2VS2QES, SW5 2MS1T2B2VS2QES, U1 4028

Commit message: Fixed LED ordering
Other:
- company: (none) -> André Fiedler <mail@andrefiedler.de>
- title: (none) -> 4028 Series BCD to Decimal Decoder Tester
Changed lines of the file:
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@@
 	(generator_version "9.0")
 	(paper "A4")
+	(title_block
+		(title "4028 Series BCD to Decimal Decoder Tester")
+		(date "2025-07-20")
+		(rev "v1.0")
+		(company "André Fiedler <mail@andrefiedler.de>")
+	)
 	(junction
 		(at 160.02 97.79)
